File: PCBs/SlaveNodePCB/SlaveNodePCB.kicad_pcb (KiCad board)
At the start: 2 copper layers, 50 x 51.6 mm, 31 parts, among them J1 8P8C, J2 Screw_Terminal_01x02, J3 Conn_01x04, J4 Conn_01x07, J5 Conn_01x03, Q1 IRLZ44N, SW1 RST, U1 AP2112K-3.3, U2 MAX485E, U3 STM8S003F3P

Commit message: Current Slave PCB
Parts:
- J2: footprint TerminalBlock_Phoenix:TerminalBlock_Phoenix_PTSM-0,5-2-2.5-V-THR_1x02_P2.50mm_Vertical -> TerminalBlock_Phoenix:TerminalBlock_Phoenix_MKDS-1,5-2-5.08_1x02_P5.08mm_Horizontal
- L1: footprint Inductor_SMD:L_6.3x6.3_H3 -> Inductor_SMD:L_Changjiang_FNR8040S
- moved L1 0.80 mm to (162.2, 66.2)
- turned J2 to 45 degrees
Routing:
- net +5V: track 112.6 -> 125.7 mm
- net /NRST: track 32.8 -> 39.5 mm
- net Net-(MP1584EN1-FB): track 0.00 -> 5.79 mm
- net GND: track 3.86 -> 0.00 mm
- net Net-(J2-Pin_1): track 36.0 -> 32.9 mm
- net +24V: track 50.0 -> 51.0 mm
- net +3.3V: track 82.6 -> 83.1 mm
- added copper zone on B.Cu, net GND
Other:
- board size 50 x 51.6 mm -> 50 x 53.8 mm
